File: LifeDetection3/LifeDetection3.kicad_pcb (KiCad board)
At the start: 2 copper layers, 101.6 x 53.3 mm, 13 parts, among them J1 Power, J2 PWM, J3 Analog, J4 PWM, J5 Analog, J6 Communication, J7 Digital

Commit message: progress
Parts:
- removed MH1, MH2, MH3, MH4, MH5, MH6: MountingHole_3.2mm, Arduino_MountingHole:MountingHole_3.2mm
- added Dr1L1: Conn_01x08, Connector_PinSocket_2.54mm:PinSocket_1x08_P2.54mm_Vertical, F.Cu at (143.2, 64.4)
- added Dr1R1: Conn_01x08, Connector_PinSocket_2.54mm:PinSocket_1x08_P2.54mm_Vertical, F.Cu at (155.9, 64.4)
- added Dr2L1: Conn_01x08, Connector_PinSocket_2.54mm:PinSocket_1x08_P2.54mm_Vertical, F.Cu at (171.1, 64.4)
- added Dr2R1: Conn_01x08, Connector_PinSocket_2.54mm:PinSocket_1x08_P2.54mm_Vertical, F.Cu at (183.8, 64.4)
- added FlapSrvo1: Conn_01x03, Connector_PinSocket_2.54mm:PinSocket_1x03_P2.54mm_Vertical, F.Cu at (140.6, 41.6)
- added J13: XT60PW-M, XT60:AMASS_XT60PW-M, F.Cu at (105.1, 69.5)
- added LSwitchD1: Conn_01x02, Connector_PinSocket_2.54mm:PinSocket_1x02_P2.54mm_Vertical, F.Cu at (188.9, 31.4)
- added LSwitchGND1: Conn_01x02, Connector_PinSocket_2.54mm:PinSocket_1x02_P2.54mm_Vertical, F.Cu at (188.9, 41.6)
- added RelayL1: Conn_01x03, Connector_PinSocket_2.54mm:PinSocket_1x03_P2.54mm_Vertical, F.Cu at (153.3, 34.0)
- added RelayR1: Conn_01x03, Connector_PinSocket_2.54mm:PinSocket_1x03_P2.54mm_Vertical, F.Cu at (163.5, 34.0)
- added Stepper1: Conn_01x04, Connector_PinSocket_2.54mm:PinSocket_1x04_P2.54mm_Vertical, F.Cu at (158.4, 105.1)
- added Stepper2: Conn_01x04, Connector_PinSocket_2.54mm:PinSocket_1x04_P2.54mm_Vertical, F.Cu at (181.3, 105.1)
Routing:
- net +5V: track 0.00 -> 132.6 mm
- net GND: track 0.00 -> 74.4 mm
- net Net-(Stepper1-Pad1): track 0.00 -> 40.8 mm
- net /*13: track 0.00 -> 39.8 mm
- net Net-(Stepper1-Pad2): track 0.00 -> 39.0 mm
- net Net-(Stepper1-Pad3): track 0.00 -> 38.1 mm
- net /*12: track 0.00 -> 37.9 mm
- net Net-(Stepper2-Pad1): track 0.00 -> 37.6 mm
- net Net-(Stepper1-Pad4): track 0.00 -> 35.2 mm
- net Net-(Stepper2-Pad2): track 0.00 -> 35.1 mm
- net Net-(Stepper2-Pad3): track 0.00 -> 34.2 mm
- net Net-(Stepper2-Pad4): track 0.00 -> 31.5 mm
- net /*9: track 0.00 -> 28.4 mm
- net /*8: track 0.00 -> 8.04 mm
Other:
- board outline removed
- copper layers 2 -> 4
- board text removed: "ICSP"
