File: LifeDetection3/LifeDetection3.kicad_pcb (KiCad board)
At the start: 2 copper layers, 101.6 x 83.8 mm, 27 parts, among them J1 Power, J12 XT60PW-M, J2 PWM, J3 Analog, J4 PWM, J5 Analog, J6 Communication, J7 Digital, P10 CONN_01X01, P8 CONN_01X01, P9 CONN_01X01, U1 TLP3545

Commit message: more final touches
Parts:
- removed the ? at (182.5, 87.3)
- removed the ? at (107.6, 87.3)
- removed P10, P8, P9: CONN_01X01, Socket_Arduino_Mega:Arduino_1pin
- removed U1: TLP3545, Package_DIP:DIP-6_W7.62mm
- added ?: , , F.Cu at (158.6, 131.1)
- added ?: , , F.Cu at (189.0, 136.1)
- added ?: , , F.Cu at (107.8, 87.9)
- added ?: , , F.Cu at (182.7, 87.9)
- added R1: ERJ-1TNF1240U, ERJ-1TNF1240U(2):RESC6432X70N, F.Cu at (143.2, 74.6)
- added Relay: TLP3545, Package_DIP:DIP-6_W7.62mm, F.Cu at (152.1, 74.6)
- renumbered Dr1L1 to Dr1L, Dr1R1 to Dr1R, Dr2L1 to Dr2L, Dr2R1 to Dr2R, FlapSrvo1 to FlapSrvo, LSwitchD1 to LSwitch, LSwitchGND1 to LSwitchGND, Vacuum+1 to Vacuum+, VacuumGND1 to VacuumGND
Routing:
- net GND: track 188.7 -> 117.9 mm, vias 2 -> 0
- net +5V: track 221.2 -> 282.6 mm, vias 3 -> 5
- net /*9: track 25.6 -> 0.00 mm
- net Net-(U1-Pad1): track 0.00 -> 5.87 mm
- net Net-(Dr1R1-Pad1): track 110.7 -> 108.7 mm
Other:
- board size 101.6 x 83.8 mm -> 104.1 x 83.8 mm
