File: LifeDetection3/LifeDetection3.kicad_sch (KiCad schematic)
At the start: 7 parts, among them J1 Power, J2 PWM, J3 Analog, J4 PWM, J5 Analog, J6 Communication, J7 Digital

Commit message: progress
Parts:
- added Dr1L1, Dr1R1, Dr2L1, Dr2R1: Conn_01x08, Connector_PinSocket_2.54mm:PinSocket_1x08_P2.54mm_Vertical, symbol Connector_Generic:Conn_01x08
- added FlapSrvo1, RelayL1, RelayR1: Conn_01x03, Connector_PinSocket_2.54mm:PinSocket_1x03_P2.54mm_Vertical, symbol Connector_Generic:Conn_01x03
- added J12: XT60PW-M, XT60:AMASS_XT60PW-M, symbol XT60PW-M:XT60PW-M
- added LSwitchD1, LSwitchGND1: Conn_01x02, Connector_PinSocket_2.54mm:PinSocket_1x02_P2.54mm_Vertical, symbol Connector_Generic:Conn_01x02
- added Stepper1, Stepper2: Conn_01x04, Connector_PinSocket_2.54mm:PinSocket_1x04_P2.54mm_Vertical, symbol Connector_Generic:Conn_01x04
Connections:
- net *10: now also Dr2L1.8 (Pin_8)
- net *11: now also Dr2L1.7 (Pin_7)
- net *12: now also Dr1L1.8 (Pin_8)
- net *13: now also Dr1L1.7 (Pin_7)
- net *8: now also FlapSrvo1.1 (Pin_1)
- net *9: now also RelayL1.1 (Pin_1)
- net +5V: now also Dr1L1.2 (Pin_2), Dr1L1.4 (Pin_4), Dr1R1.7 (Pin_7), Dr2L1.2 (Pin_2), Dr2L1.4 (Pin_4), Dr2R1.7 (Pin_7), FlapSrvo1.2 (Pin_2), RelayL1.2 (Pin_2), RelayL1.3 (Pin_3)
- net 47: now also LSwitchD1.2 (Pin_2)
- net 48: now also LSwitchD1.1 (Pin_1)
- net GND: now also Dr1L1.3 (Pin_3), Dr1R1.8 (Pin_8), Dr2L1.3 (Pin_3), Dr2R1.8 (Pin_8), FlapSrvo1.3 (Pin_3), LSwitchGND1.1 (Pin_1), LSwitchGND1.2 (Pin_2)
- new net: Dr1R1.1 (Pin_1), Dr2R1.1 (Pin_1), J12.2 (-), RelayR1.2 (Pin_2)
- new net: Dr1R1.2 (Pin_2), Dr2R1.2 (Pin_2), J12.1 (+)
- new net: Dr2R1.3 (Pin_3), Stepper2.1 (Pin_1)
- new net: Dr2R1.4 (Pin_4), Stepper2.2 (Pin_2)
- new net: Dr2R1.5 (Pin_5), Stepper2.3 (Pin_3)
- new net: Dr2R1.6 (Pin_6), Stepper2.4 (Pin_4)
- new net: Dr1R1.3 (Pin_3), Stepper1.1 (Pin_1)
- new net: Dr1R1.4 (Pin_4), Stepper1.2 (Pin_2)
- new net: Dr1R1.5 (Pin_5), Stepper1.3 (Pin_3)
- new net: Dr1R1.6 (Pin_6), Stepper1.4 (Pin_4)
Other:
- moved on the sheet: J1, J2, J3, J4, J5, J6, J7

Commit message: 2 layers + connector footprint
Parts:
- J12: footprint XT60:AMASS_XT60PW-M -> XT60PW-M:AMASS_XT60PW-M
Changed lines of the file:
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@@
       (effects (font (size 1.27 1.27)) (justify left))
     )
-    (property "Footprint" "XT60:AMASS_XT60PW-M" (id 2) (at 80.01 110.49 0)
+    (property "Footprint" "XT60PW-M:AMASS_XT60PW-M" (id 2) (at 80.01 110.49 0)
       (effects (font (size 1.27 1.27)) (justify bottom) hide)
     )
@@
     )
     (path "/f4ec02f2-00d2-4de8-8e6f-e4d175a632ad"
-      (reference "J12") (unit 1) (value "XT60PW-M") (footprint "XT60:AMASS_XT60PW-M")
+      (reference "J12") (unit 1) (value "XT60PW-M") (footprint "XT60PW-M:AMASS_XT60PW-M")
     )
     (path "/8b0cbbb0-2f60-4f01-a684-f0316ec4e436"

Commit message: more tracing
Parts:
- added +Batt1: Conn_01x01, TestPoint:TestPoint_THTPad_D4.0mm_Drill2.0mm, symbol Connector_Generic:Conn_01x01
- added TempSens1: Conn_01x04, Connector_PinSocket_2.54mm:PinSocket_1x04_P2.54mm_Vertical, symbol Connector_Generic:Conn_01x04
Connections:
- net +3V3: now also TempSens1.3 (Pin_3)
- net GND: now also TempSens1.4 (Pin_4)
- net SCL/21: now also TempSens1.1 (Pin_1)
- net SDA/20: now also TempSens1.2 (Pin_2)
- net at Dr1R1.2 (Pin_2), Dr2R1.2 (Pin_2), J12.1 (+): now also +Batt1.1 (Pin_1)
Changed lines of the file:
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@@
   (junction (at 85.09 54.61) (diameter 0) (color 0 0 0 0)
   )
+  (junction (at 85.09 39.37) (diameter 0) (color 0 0 0 0)
+  )
   (junction (at 67.31 64.77) (diameter 0) (color 0 0 0 0)
   )
+  (junction (at 234.95 25.4) (diameter 0) (color 0 0 0 0)
+  )
   (junction (at 77.47 80.01) (diameter 0) (color 0 0 0 0)
   )
@@
   )
   (junction (at 24.13 67.31) (diameter 0) (color 0 0 0 0)
+  )
+  (junction (at 69.85 101.6) (diameter 0) (color 0 0 0 0)
   )
   (junction (at 278.13 115.57) (diameter 1.016) (color 0 0 0 0)
@@
     (stroke (width 0) (type solid) (color 0 0 0 0))
   )
+  (wire (pts (xy 106.68 25.4) (xy 234.95 25.4))
+    (stroke (width 0) (type default) (color 0 0 0 0))
+  )
   (wire (pts (xy 265.43 33.02) (xy 278.13 33.02))
     (stroke (width 0) (type solid) (color 0 0 0 0))
   )
-  (wire (pts (xy 234.95 22.86) (xy 234.95 35.56))
+  (wire (pts (xy 234.95 22.86) (xy 234.95 25.4))
     (stroke (width 0) (type solid) (color 0 0 0 0))
   )
@@
     (stroke (width 0) (type solid) (color 0 0 0 0))
   )
+  (wire (pts (xy 121.92 34.29) (xy 127 34.29))
+    (stroke (width 0) (type default) (color 0 0 0 0))
+  )
   (wire (pts (xy 265.43 35.56) (xy 278.13 35.56))
     (stroke (width 0) (type solid) (color 0 0 0 0))
@@
     (stroke (width 0) (type default) (color 0 0 0 0))
   )
+  (wire (pts (xy 69.85 101.6) (xy 87.63 101.6))
+    (stroke (width 0) (type default) (color 0 0 0 0))
+  )
   (wire (pts (xy 265.43 93.98) (xy 278.13 93.98))
     (stroke (width 0) (type solid) (color 0 0 0 0))
@@
     (stroke (width 0) (type default) (color 0 0 0 0))
   )
+  (wire (pts (xy 69.85 101.6) (xy 69.85 67.31))
+    (stroke (width 0) (type default) (color 0 0 0 0))
+  )
   (wire (pts (xy 16.51 69.85) (xy 31.75 69.85))
     (stroke (width 0) (type default) (color 0 0 0 0))
@@
     (stroke (width 0) (type default) (color 0 0 0 0))
   )
+  (wire (pts (xy 234.95 25.4) (xy 234.95 35.56))
+    (stroke (width 0) (type solid) (color 0 0 0 0))
+  )
+  (wire (pts (xy 106.68 36.83) (xy 127 36.83))
+    (stroke (width 0) (type default) (color 0 0 0 0))
+  )
   (wire (pts (xy 237.49 60.96) (xy 224.79 60.96))
     (stroke (width 0) (type solid) (color 0 0 0 0))
@@
     (stroke (width 0) (type solid) (color 0 0 0 0))
   )
-  (wire (pts (xy 85.09 26.67) (xy 85.09 54.61))
+  (wire (pts (xy 85.09 26.67) (xy 85.09 39.37))
     (stroke (width 0) (type default) (color 0 0 0 0))
   )
@@
     (stroke (width 0) (type default) (color 0 0 0 0))
   )
+  (wire (pts (xy 85.09 39.37) (xy 85.09 54.61))
+    (stroke (width 0) (type default) (color 0 0 0 0))
+  )
   (wire (pts (xy 77.47 57.15) (xy 111.76 57.15))
     (stroke (width 0) (type default) (color 0 0 0 0))
@@
     (stroke (width 0) (type solid) (color 0 0 0 0))
   )
+  (wire (pts (xy 121.92 31.75) (xy 127 31.75))
+    (stroke (width 0) (type default) (color 0 0 0 0))
+  )
   (wire (pts (xy 232.41 105.41) (xy 232.41 115.57))
     (stroke (width 0) (type solid) (color 0 0 0 0))
@@
     (stroke (width 0) (type default) (color 0 0 0 0))
   )
+  (wire (pts (xy 106.68 25.4) (xy 106.68 36.83))
+    (stroke (width 0) (type default) (color 0 0 0 0))
+  )
   (wire (pts (xy 57.15 64.77) (xy 67.31 64.77))
     (stroke (width 0) (type default) (color 0 0 0 0))
@@
     (stroke (width 0) (type solid) (color 0 0 0 0))
   )
-  (wire (pts (xy 69.85 107.95) (xy 69.85 67.31))
+  (wire (pts (xy 69.85 107.95) (xy 69.85 101.6))
     (stroke (width 0) (type default) (color 0 0 0 0))
   )
@@
     (stroke (width 0) (type default) (color 0 0 0 0))
   )
+  (wire (pts (xy 85.09 39.37) (xy 127 39.37))
+    (stroke (width 0) (type default) (color 0 0 0 0))
+  )
   (wire (pts (xy 265.43 96.52) (xy 278.13 96.52))
     (stroke (width 0) (type solid) (color 0 0 0 0))
@@
     (effects (font (size 1.27 1.27)) (justify left bottom))
   )
+  (label "SCL{slash}21" (at 121.92 31.75 0)
+    (effects (font (size 1.27 1.27)) (justify left bottom))
+  )
   (label "A2" (at 224.79 60.96 0)
     (effects (font (size 1.27 1.27)) (justify left bottom))
@@
   (label "TX2{slash}16" (at 278.13 86.36 180)
     (effects (font (size 1.27 1.27)) (justify right bottom))
+  )
+  (label "SDA{slash}20" (at 121.92 34.29 0)
+    (effects (font (size 1.27 1.27)) (justify left bottom))
   )
   (label "*5" (at 278.13 60.96 180)
@@
     (pin "2")
   )
+  (symbol (lib_id "Connector_Generic:Conn_01x01") (at 92.71 101.6 0) (unit 1)
+    (in_bom yes) (on_board yes) (fields_autoplaced)
+    (property "Reference" "+Batt1" (id 0) (at 95.25 100.3299 0)
+      (effects (font (size 1.27 1.27)) (justify left))
+    )
+    (property "Value" "Conn_01x01" (id 1) (at 95.25 102.8699 0)
+      (effects (font (size 1.27 1.27)) (justify left))
+    )
+    (property "Footprint" "TestPoint:TestPoint_THTPad_D4.0mm_Drill2.0mm" (id 2) (at 92.71 101.6 0)
+      (effects (font (size 1.27 1.27)) hide)
+    )
+    (property "Datasheet" "~" (id 3) (at 92.71 101.6 0)
+      (effects (font (size 1.27 1.27)) hide)
+    )
+    (pin "1")
+  )
   (symbol (lib_id "power:VCC") (at 229.87 22.86 0) (unit 1)
     (in_bom yes) (on_board yes)
@@
     (pin "1")
   )
+  (symbol (lib_id "Connector_Generic:Conn_01x04") (at 132.08 34.29 0) (unit 1)
+    (in_bom yes) (on_board yes) (fields_autoplaced)
+    (property "Reference" "TempSens1" (id 0) (at 134.62 34.2899 0)
+      (effects (font (size 1.27 1.27)) (justify left))
+    )
+    (property "Value" "Conn_01x04" (id 1) (at 134.62 36.8299 0)
+      (effects (font (size 1.27 1.27)) (justify left))
+    )
+    (property "Footprint" "Connector_PinSocket_2.54mm:PinSocket_1x04_P2.54mm_Vertical" (id 2) (at 132.08 34.29 0)
+      (effects (font (size 1.27 1.27)) hide)
+    )
+    (property "Datasheet" "~" (id 3) (at 132.08 34.29 0)
+      (effects (font (size 1.27 1.27)) hide)
+    )
+    (pin "1")
+    (pin "2")
+    (pin "3")
+    (pin "4")
+  )
   (symbol (lib_id "Connector_Generic:Conn_01x08") (at 52.07 44.45 0) (mirror y) (unit 1)
     (in_bom yes) (on_board yes) (fields_autoplaced)
@@
       (reference "#PWR0104") (unit 1) (value "GND") (footprint "")
     )
+    (path "/5924eeaa-d3bc-4557-ada7-671e5c92afce"
+      (reference "+Batt1") (unit 1) (value "Conn_01x01") (footprint "TestPoint:TestPoint_THTPad_D4.0mm_Drill2.0mm")
+    )
     (path "/094473b1-1ad7-4da9-82fe-a8d474c45d8b"
       (reference "Dr1L1") (unit 1) (value "Conn_01x08") (footprint "Connector_PinSocket_2.54mm:PinSocket_1x08_P2.54mm_Vertical")
@@
       (reference "Stepper2") (unit 1) (value "Conn_01x04") (footprint "Connector_PinSocket_2.54mm:PinSocket_1x04_P2.54mm_Vertical")
     )
-  )
+    (path "/d7a730fe-28d4-40b8-91fc-a252cfbdcda3"
+      (reference "TempSens1") (unit 1) (value "Conn_01x04") (footprint "Connector_PinSocket_2.54mm:PinSocket_1x04_P2.54mm_Vertical")
+    )
+  )
