File: LifeDetection3/LifeDetection3.kicad_sch (KiCad schematic)
At the start: 21 parts, among them J1 Power, J12 XT60PW-M, J2 PWM, J3 Analog, J4 PWM, J5 Analog, J6 Communication, J7 Digital, U1 TLP3545

Commit message: more final touches
Connections:
- net *9: no longer U1.4 (DRAIN)
- net +5V: no longer U1.6 (DRAIN)
- net GND: now also U1.2 (CATHODE); no longer U1.5 (SOURCE)
- net at Dr1R1.1 (Pin_1), Dr2R1.1 (Pin_1), J12.2 (-): now also U1.5 (SOURCE)
- net at VacuumGND1.1 (Pin_1): now also U1.6 (DRAIN)
Other:
- company: (none) -> Designed by: Maxime Couture & Yadah Ngolo
- title: (none) -> Life Detection Shield Mk.1
- moved on the sheet: VacuumGND1

Commit message: stuff
Parts:
- added R1: ERJ-1TNF1240U, ERJ-1TNF1240U(2):RESC6432X70N, symbol ERJ-1TNF1240U:ERJ-1TNF1240U
Connections:
- net +5V: now also R1.1
- net at U1.1 (ANODE): now also R1.2
Changed lines of the file:
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@@
     (stroke (width 0) (type solid) (color 0 0 0 0))
-  )
-  (wire (pts (xy 114.3254 63.5) (xy 123.1646 63.5))
-    (stroke (width 0) (type default) (color 0 0 0 0))
   )
   (wire (pts (xy 77.47 80.01) (xy 123.19 80.01))
@@
     (stroke (width 0) (type default) (color 0 0 0 0))
   )
-  (wire (pts (xy 100.33 60.96) (xy 114.3254 60.96))
-    (stroke (width 0) (type default) (color 0 0 0 0))
-  )
   (wire (pts (xy 67.31 118.11) (xy 67.31 110.49))
     (stroke (width 0) (type default) (color 0 0 0 0))
@@
     (stroke (width 0) (type solid) (color 0 0 0 0))
   )
-  (wire (pts (xy 114.3254 63.5) (xy 114.3254 60.96))
-    (stroke (width 0) (type default) (color 0 0 0 0))
-  )
   (wire (pts (xy 265.43 27.94) (xy 278.13 27.94))
     (stroke (width 0) (type solid) (color 0 0 0 0))
@@
   (label "TX3{slash}14" (at 278.13 81.28 180)
     (effects (font (size 1.27 1.27)) (justify right bottom))
-  )
-  (label "*9" (at 100.33 60.96 0)
-    (effects (font (size 1.27 1.27)) (justify left bottom))
   )
   (label "32" (at 257.81 105.41 270)
@@
     (pin "4")
   )
+  (symbol (lib_id "ERJ-1TNF1240U:ERJ-1TNF1240U") (at 125.73 53.34 0) (unit 1)
+    (in_bom yes) (on_board yes) (fields_autoplaced)
+    (property "Reference" "R1" (id 0) (at 125.73 45.72 0))
+    (property "Value" "ERJ-1TNF1240U" (id 1) (at 125.73 48.26 0))
+    (property "Footprint" "ERJ-1TNF1240U(2):RESC6432X70N" (id 2) (at 125.73 53.34 0)
+      (effects (font (size 1.27 1.27)) (justify left bottom) hide)
+    )
+    (property "Datasheet" "" (id 3) (at 125.73 53.34 0)
+      (effects (font (size 1.27 1.27)) (justify left bottom) hide)
+    )
+    (pin "1")
+    (pin "2")
+  )
   (symbol (lib_id "2023-02-05_19-50-21:TLP3545") (at 144.78 52.07 0) (unit 1)
     (in_bom yes) (on_board yes) (fields_autoplaced)
@@
       (reference "LSwitchGND1") (unit 1) (value "Conn_01x02") (footprint "Connector_PinSocket_2.54mm:PinSocket_1x02_P2.54mm_Vertical")
     )
+    (path "/a66e1df5-8625-47e8-9676-94bef11bec30"
+      (reference "R1") (unit 1) (value "ERJ-1TNF1240U") (footprint "ERJ-1TNF1240U(2):RESC6432X70N")
+    )
     (path "/3ac3779e-71a1-4d79-9194-d968fa92e89d"
